File: A600_68k_PLCC_to_DIP64 _v1.sch (KiCad schematic (older format))
At the start: 7 parts, among them U1 MC68000_PLCC68, U2 68000_SOCKET

Commit message: Updated to Rev B
Re-routed 4-layer design.
Parts:
- added C1, C2, C3, C4, C5: 100nf, Capacitor_SMD:C_0805_2012Metric_Pad1.18x1.45mm_HandSolder, symbol Device:C
- added J1: 171826-4, A600 68k PLCC to DIP64:TE_171826-4, symbol 171826-4:171826-4
- R1, R2: footprint Resistor_SMD:R_0805_2012Metric_Pad1.15x1.40mm_HandSolder -> Resistor_SMD:R_0805_2012Metric_Pad1.20x1.40mm_HandSolder
- U2: symbol MC68000_DIP64_SOCKET:68000_SOCKET -> 68000_DIP_SOCKET:68000_SOCKET
Connections:
- net labels removed: e, fc0, fc1, fc2, ~bg, ~vma
- wire segments 190 -> 209
- no-connect marks 3 -> 14
Other:
- moved on the sheet: H1, H2, H3

Commit message: Corrected cap values
Parts:
- C1, C2, C3, C4, C5: value 100nf -> 10uf
Changed lines of the file:
@@
 P 800 7050
 F 0 "C1" H 915 7096 50  0000 L CNN
-F 1 "100nf" H 915 7005 50  0000 L CNN
+F 1 "10uf" H 915 7005 50  0000 L CNN
 F 2 "Capacitor_SMD:C_0805_2012Metric_Pad1.18x1.45mm_HandSolder" H 838 6900 50  0001 C CNN
 F 3 "~" H 800 7050 50  0001 C CNN
@@
 P 1250 7050
 F 0 "C2" H 1365 7096 50  0000 L CNN
-F 1 "100nf" H 1365 7005 50  0000 L CNN
+F 1 "10uf" H 1365 7005 50  0000 L CNN
 F 2 "Capacitor_SMD:C_0805_2012Metric_Pad1.18x1.45mm_HandSolder" H 1288 6900 50  0001 C CNN
 F 3 "~" H 1250 7050 50  0001 C CNN
@@
 P 1700 7050
 F 0 "C3" H 1815 7096 50  0000 L CNN
-F 1 "100nf" H 1815 7005 50  0000 L CNN
+F 1 "10uf" H 1815 7005 50  0000 L CNN
 F 2 "Capacitor_SMD:C_0805_2012Metric_Pad1.18x1.45mm_HandSolder" H 1738 6900 50  0001 C CNN
 F 3 "~" H 1700 7050 50  0001 C CNN
@@
 P 2150 7050
 F 0 "C4" H 2265 7096 50  0000 L CNN
-F 1 "100nf" H 2265 7005 50  0000 L CNN
+F 1 "10uf" H 2265 7005 50  0000 L CNN
 F 2 "Capacitor_SMD:C_0805_2012Metric_Pad1.18x1.45mm_HandSolder" H 2188 6900 50  0001 C CNN
 F 3 "~" H 2150 7050 50  0001 C CNN
@@
 P 2600 7050
 F 0 "C5" H 2715 7096 50  0000 L CNN
-F 1 "100nf" H 2715 7005 50  0000 L CNN
+F 1 "10uf" H 2715 7005 50  0000 L CNN
 F 2 "Capacitor_SMD:C_0805_2012Metric_Pad1.18x1.45mm_HandSolder" H 2638 6900 50  0001 C CNN
 F 3 "~" H 2600 7050 50  0001 C CNN
